Commit message: feature: keyboard_driver for manual control

File: src/go_car_description/urdf/include/gazebo.xacro (robot description, xacro)
@@ -51,51 +51,6 @@
     <maxVel>10.0</maxVel>
   </gazebo>
-  <!-- Actuators definition -->
-  <transmission name="rear_left_wheel_gearing">
-    <type>transmission_interface/SimpleTransmission</type>
-    <joint name="chassis_to_rear_left_wheel">
-      <hardwareInterface>hardware_interface/EffortJointInterface</hardwareInterface>
-    </joint>
-    <actuator name="traction_motor_left">
-      <hardwareInterface>hardware_interface/EffortJointInterface</hardwareInterface>
-      <mechanicalReduction>1</mechanicalReduction>
-    </actuator>
-  </transmission>
-  <transmission name="rear_right_wheel_gearing">
-    <type>transmission_interface/SimpleTransmission</type>
-    <joint name="chassis_to_rear_right_wheel">
-      <hardwareInterface>hardware_interface/EffortJointInterface</hardwareInterface>
-    </joint>
-    <actuator name="traction_motor_right">
-      <hardwareInterface>hardware_interface/EffortJointInterface</hardwareInterface>
-      <mechanicalReduction>1</mechanicalReduction>
-    </actuator>
-  </transmission>
-  <transmission name="left_steering_gearing">
-    <type>transmission_interface/SimpleTransmission</type>
-    <joint name="base_to_left_steering_column">
-      <hardwareInterface>hardware_interface/EffortJointInterface</hardwareInterface>
-    </joint>
-    <actuator name="left_steering_servo">
-      <hardwareInterface>hardware_interface/EffortJointInterface</hardwareInterface>
-      <mechanicalReduction>1</mechanicalReduction>
-    </actuator>
-  </transmission>
-  <transmission name="right_steering_gearing">
-    <type>transmission_interface/SimpleTransmission</type>
-    <joint name="base_to_right_steering_column">
-      <hardwareInterface>hardware_interface/EffortJointInterface</hardwareInterface>
-    </joint>
-    <actuator name="right_steering_servo">
-      <hardwareInterface>hardware_interface/EffortJointInterface</hardwareInterface>
-      <mechanicalReduction>1</mechanicalReduction>
-    </actuator>
-  </transmission>
   <!-- Plugins -->
   <gazebo>
-    <!-- <plugin name="gazebo_ros_control" filename="libgazebo_ros_control.so">
-      <robotNamespace>/$(arg robot_name)</robotNamespace>
-      <robotSimType>gazebo_ros_control/DefaultRobotHWSim</robotSimType>
-    </plugin> -->
     <plugin name="ackermann_control_plugin" filename="libackermann_control_plugin.so"/>
     <plugin filename="libgazebo_ros_joint_state_publisher.so" name="joint_state_publisher">
