Commit message: Asymetric steering bug solved

File: src/go_car_description/urdf/go_car_model.xacro (robot description, xacro)
@@ -17,5 +17,5 @@
     <axis xyz="0.0 0.0 1"/>
     <origin xyz="${distanceX_CM_to_front_wheel_axis} ${distanceY_CM_to_wheel_center} ${distanceZ_CM_to_wheel_center}" rpy="0.0 0.0 0.0"/>
-    <limit lower="${-5/9*pi/5}" upper="${5/9*pi/5}" effort="25000" velocity="5"/>
+    <limit lower="${-5/9*pi/2}" upper="${5/9*pi/2}" effort="15000" velocity="0.25"/>
   </joint>
   <joint name="base_to_right_steering_column" type="revolute">
@@ -24,5 +24,5 @@
     <axis xyz="0.0 0.0 1"/>
     <origin xyz="${distanceX_CM_to_front_wheel_axis} ${-distanceY_CM_to_wheel_center} ${distanceZ_CM_to_wheel_center}" rpy="0.0 0.0 0.0"/>
-    <limit lower="${-5/9*pi/2}" upper="${5/9*pi/2}" effort="25000" velocity="5"/>
+    <limit lower="${-5/9*pi/2}" upper="${5/9*pi/2}" effort="15000" velocity="0.25"/>
   </joint>
   <joint name="base_to_chassis" type="fixed">

Commit message: feature: Major progress in low level control of car

File: src/go_car_description/urdf/go_car_model.xacro (robot description, xacro)
@@ -7,9 +7,4 @@
   <!-- First tf level -->
   <link name="base_link"/>
-  <joint name="base_to_base_footprint" type="fixed">
-    <parent link="base_link"/>
-    <child link="base_footprint"/>
-    <origin xyz="0.0 0.0 ${distanceZ_CM_to_ground}" rpy="0.0 0.0 0.0"/>
-  </joint>
   <joint name="base_to_left_steering_column" type="revolute">
     <parent link="base_link"/>
@@ -32,5 +27,4 @@
   </joint>
   <!-- Second tf level -->
-  <link name="base_footprint"/>
   <xacro:insert_block name="chassis_link"/>
   <joint name="chassis_to_rear_left_wheel" type="continuous">
@@ -39,5 +33,5 @@
     <origin xyz="${distanceX_CM_to_rear_wheel_axis} ${distanceY_CM_to_wheel_center} ${distanceZ_CM_to_wheel_center}" rpy="0.0 0.0 0.0"/>
     <axis xyz="0.0 1.0 0.0"/>
-    <limit effort="500" velocity="200"/>
+    <limit effort="5000" velocity="200"/>
   </joint>
   <joint name="chassis_to_rear_right_wheel" type="continuous">
@@ -46,5 +40,5 @@
     <origin xyz="${distanceX_CM_to_rear_wheel_axis} ${-distanceY_CM_to_wheel_center} ${distanceZ_CM_to_wheel_center}" rpy="0.0 0.0 0.0"/>
     <axis xyz="0.0 1.0 0.0"/>
-    <limit effort="500" velocity="200"/>
+    <limit effort="5000" velocity="200"/>
   </joint>
   <xacro:steering_column_link RL="left"/>
@@ -54,5 +48,5 @@
     <child link="front_left_wheel_link"/>
     <axis xyz="0.0 1.0 0.0"/>
-    <limit effort="500" velocity="200"/>
+    <limit effort="5000" velocity="200"/>
   </joint>
   <joint name="steering_column_to_front_right_wheel" type="continuous">
@@ -60,5 +54,5 @@
     <child link="front_right_wheel_link"/>
     <axis xyz="0.0 1.0 0.0"/>
-    <limit effort="500" velocity="200"/>
+    <limit effort="5000" velocity="200"/>
   </joint>
   <!-- Third tf level -->

File: src/go_car_description/urdf/include/gazebo.xacro (robot description, xacro)
@@ -3,6 +3,6 @@
   <!-- Friction parameters -->
   <gazebo reference="rear_right_wheel_link">
-    <mu1>10000000</mu1>
-    <mu2>10000000</mu2>
+    <mu1>1</mu1>
+    <mu2>1</mu2>
     <kp>10000000</kp>
     <kd>1</kd>
@@ -11,6 +11,6 @@
   </gazebo>
   <gazebo reference="rear_left_wheel_link">
-    <mu1>10000000</mu1>
-    <mu2>10000000</mu2>
+    <mu1>1</mu1>
+    <mu2>1</mu2>
     <kp>10000000</kp>
     <kd>1</kd>
@@ -19,6 +19,6 @@
   </gazebo>
   <gazebo reference="front_right_wheel_link">
-    <mu1>10000000</mu1>
-    <mu2>10000000</mu2>
+    <mu1>1</mu1>
+    <mu2>1</mu2>
     <kp>10000000</kp>
     <kd>1</kd>
@@ -27,6 +27,6 @@
   </gazebo>
   <gazebo reference="front_left_wheel_link">
-    <mu1>10000000</mu1>
-    <mu2>10000000</mu2>
+    <mu1>1</mu1>
+    <mu2>1</mu2>
     <kp>10000000</kp>
     <kd>1</kd>
@@ -94,12 +94,11 @@
   <!-- Plugins -->
   <gazebo>
-    <plugin name="gazebo_ros_control" filename="libgazebo_ros_control.so">
+    <!-- <plugin name="gazebo_ros_control" filename="libgazebo_ros_control.so">
       <robotNamespace>/$(arg robot_name)</robotNamespace>
       <robotSimType>gazebo_ros_control/DefaultRobotHWSim</robotSimType>
-    </plugin>
-  </gazebo>
-  <gazebo>
+    </plugin> -->
+    <plugin name="ackermann_control_plugin" filename="libackermann_control_plugin.so"/>
     <plugin filename="libgazebo_ros_joint_state_publisher.so" name="joint_state_publisher">
-      <jointName>steering_column_to_front_left_wheel, steering_column_to_front_right_wheel</jointName>
+      <jointName>chassis_to_rear_left_wheel, chassis_to_rear_right_wheel, base_to_left_steering_column, base_to_right_steering_column</jointName>
       <updateRate>50.0</updateRate>
       <robotNamespace>/$(arg robot_name)</robotNamespace>

Commit message: feature: city world + steering improvement

File: src/go_car_description/urdf/go_car_model.xacro (robot description, xacro)
@@ -12,5 +12,5 @@
     <axis xyz="0.0 0.0 1"/>
     <origin xyz="${distanceX_CM_to_front_wheel_axis} ${distanceY_CM_to_wheel_center} ${distanceZ_CM_to_wheel_center}" rpy="0.0 0.0 0.0"/>
-    <limit lower="${-5/9*pi/2}" upper="${5/9*pi/2}" effort="15000" velocity="0.25"/>
+    <limit lower="${-6/9*pi/2}" upper="${6/9*pi/2}" effort="100000" velocity="100000"/>
   </joint>
   <joint name="base_to_right_steering_column" type="revolute">
@@ -19,5 +19,5 @@
     <axis xyz="0.0 0.0 1"/>
     <origin xyz="${distanceX_CM_to_front_wheel_axis} ${-distanceY_CM_to_wheel_center} ${distanceZ_CM_to_wheel_center}" rpy="0.0 0.0 0.0"/>
-    <limit lower="${-5/9*pi/2}" upper="${5/9*pi/2}" effort="15000" velocity="0.25"/>
+    <limit lower="${-6/9*pi/2}" upper="${6/9*pi/2}" effort="100000" velocity="100000"/>
   </joint>
   <joint name="base_to_chassis" type="fixed">
@@ -33,5 +33,5 @@
     <origin xyz="${distanceX_CM_to_rear_wheel_axis} ${distanceY_CM_to_wheel_center} ${distanceZ_CM_to_wheel_center}" rpy="0.0 0.0 0.0"/>
     <axis xyz="0.0 1.0 0.0"/>
-    <limit effort="5000" velocity="200"/>
+    <limit effort="100000" velocity="100000"/>
   </joint>
   <joint name="chassis_to_rear_right_wheel" type="continuous">
@@ -40,5 +40,5 @@
     <origin xyz="${distanceX_CM_to_rear_wheel_axis} ${-distanceY_CM_to_wheel_center} ${distanceZ_CM_to_wheel_center}" rpy="0.0 0.0 0.0"/>
     <axis xyz="0.0 1.0 0.0"/>
-    <limit effort="5000" velocity="200"/>
+    <limit effort="100000" velocity="100000"/>
   </joint>
   <xacro:steering_column_link RL="left"/>
@@ -48,5 +48,5 @@
     <child link="front_left_wheel_link"/>
     <axis xyz="0.0 1.0 0.0"/>
-    <limit effort="5000" velocity="200"/>
+    <limit effort="100000" velocity="100000"/>
   </joint>
   <joint name="steering_column_to_front_right_wheel" type="continuous">
@@ -54,5 +54,5 @@
     <child link="front_right_wheel_link"/>
     <axis xyz="0.0 1.0 0.0"/>
-    <limit effort="5000" velocity="200"/>
+    <limit effort="100000" velocity="100000"/>
   </joint>
   <!-- Third tf level -->

File: src/go_car_description/urdf/include/gazebo.xacro (robot description, xacro)
@@ -35,5 +35,5 @@
   </gazebo>
   <!-- Suspension parameters -->
-  <gazebo reference="right_steering_column_link">
+  <!-- <gazebo reference="right_steering_column_link">
     <mu1>0.6</mu1>
     <mu2>0.5</mu2>
@@ -42,6 +42,6 @@
     <minDepth>0.01</minDepth>
     <maxVel>10.0</maxVel>
-  </gazebo>
-  <gazebo reference="left_steering_column_link">
+  </gazebo> -->
+  <!-- <gazebo reference="left_steering_column_link">
     <mu1>0.6</mu1>
     <mu2>0.5</mu2>
@@ -50,5 +50,5 @@
     <minDepth>0.01</minDepth>
     <maxVel>10.0</maxVel>
-  </gazebo>
+  </gazebo> -->
   <!-- Plugins -->
   <gazebo>

File: src/go_car_description/urdf/include/links.xacro (robot description, xacro)
@@ -8,5 +8,5 @@
             </inertial>
             <collision>
-                <origin xyz="0.25 0.0 0.0" rpy="0.0 0.0 0.0"/>
+                <origin xyz="0.25 0.0 0.2" rpy="0.0 0.0 0.0"/>
                 <geometry>
                     <box size="${chassis_length} ${chassis_width} ${chassis_height}"/>

File: src/go_car_description/urdf/include/params.xacro (robot description, xacro)
@@ -28,5 +28,5 @@
     <xacro:property name="str_angle" value="0.6"/>
     <xacro:property name="car_width" value="1.301"/>
-    <xacro:property name="chassis_height" value="1.5"/>
+    <xacro:property name="chassis_height" value="1.3"/>
     <xacro:property name="chassis_length" value="5"/>
     <xacro:property name="chassis_width" value="2.2"/>

Commit message: gmapping

File: src/go_car_description/urdf/go_car_model.xacro (robot description, xacro)
@@ -5,8 +5,14 @@
   <xacro:include filename="$(find go_car_description)/urdf/include/snippets.xacro"/>
   <xacro:include filename="$(find go_car_description)/urdf/include/links.xacro"/>
+  <xacro:include filename="$(find go_car_description)/urdf/include/sensors.xacro"/>
   <!-- First tf level -->
   <link name="base_link"/>
-  <joint name="base_to_left_steering_column" type="revolute">
+  <joint name="base_to_chassis" type="fixed">
     <parent link="base_link"/>
+    <child link="chassis_link"/>
+    <origin xyz="0.0 0.0 0.0" rpy="0.0 0.0 0.0"/>
+  </joint>
+  <joint name="chassis_to_left_steering_column" type="revolute">
+    <parent link="chassis_link"/>
     <child link="left_steering_column_link"/>
     <axis xyz="0.0 0.0 1"/>
@@ -14,15 +20,10 @@
     <limit lower="${-6/9*pi/2}" upper="${6/9*pi/2}" effort="100000" velocity="100000"/>
   </joint>
-  <joint name="base_to_right_steering_column" type="revolute">
-    <parent link="base_link"/>
+  <joint name="chassis_to_right_steering_column" type="revolute">
+    <parent link="chassis_link"/>
     <child link="right_steering_column_link"/>
     <axis xyz="0.0 0.0 1"/>
     <origin xyz="${distanceX_CM_to_front_wheel_axis} ${-distanceY_CM_to_wheel_center} ${distanceZ_CM_to_wheel_center}" rpy="0.0 0.0 0.0"/>
     <limit lower="${-6/9*pi/2}" upper="${6/9*pi/2}" effort="100000" velocity="100000"/>
-  </joint>
-  <joint name="base_to_chassis" type="fixed">
-    <parent link="base_link"/>
-    <child link="chassis_link"/>
-    <origin xyz="0.0 0.0 0.0" rpy="0.0 0.0 0.0"/>
   </joint>
   <!-- Second tf level -->
@@ -64,10 +65,10 @@
     <parent link="chassis_link"/>
     <child link="camera_link"/>
-    <origin xyz="0.0 0.0 1.2" rpy="0.0 0.0 0.0"/>
+    <origin xyz="0.0 0.0 0.8" rpy="0.0 0.0 0.0"/>
   </joint>
   <joint name="chassis_to_lidar" type="fixed">
     <parent link="chassis_link"/>
     <child link="lidar_link"/>
-    <origin xyz="0.0 0.0 1.4" rpy="0.0 0.0 0.0"/>
+    <origin xyz="${chassis_length/2+0.25} 0.0 -0.25" rpy="0.0 0.0 0.0"/>
   </joint>
   <!-- Gazebo -->

File: src/go_car_description/urdf/include/gazebo.xacro (robot description, xacro)
@@ -19,4 +19,12 @@
   </gazebo>
   <gazebo reference="front_right_wheel_link">
+    <mu1>1</mu1>
+    <mu2>1</mu2>
+    <kp>10000000</kp>
+    <kd>1</kd>
+    <minDepth>0.01</minDepth>
+    <maxVel>100.0</maxVel>
+  </gazebo>
+  <gazebo reference="front_left_wheel_link">
     <mu1>1</mu1>
     <mu2>1</mu2>
@@ -55,48 +63,19 @@
     <plugin name="ackermann_control_plugin" filename="libackermann_control_plugin.so"/>
     <plugin filename="libgazebo_ros_joint_state_publisher.so" name="joint_state_publisher">
-      <jointName>chassis_to_rear_left_wheel, chassis_to_rear_right_wheel, base_to_left_steering_column, base_to_right_steering_column</jointName>
+      <jointName>chassis_to_rear_left_wheel, chassis_to_rear_right_wheel, chassis_to_left_steering_column, steering_column_to_front_left_wheel, chassis_to_right_steering_column, steering_column_to_front_right_wheel</jointName>
       <updateRate>50.0</updateRate>
       <robotNamespace>/$(arg robot_name)</robotNamespace>
       <alwaysOn>true</alwaysOn>
     </plugin>
-  </gazebo>
-  <gazebo reference="camera_link">
-    <sensor type="camera" name="camera1">
-      <update_rate>30.0</update_rate>
-      <camera name="head">
-        <horizontal_fov>1.3962634</horizontal_fov>
-        <image>
-          <width>800</width>
-          <height>800</height>
-          <format>R8G8B8</format>
-        </image>
-        <clip>
-          <near>0.02</near>
-          <far>300</far>
-        </clip>
-        <noise>
-          <type>gaussian</type>
-          <!-- Noise is sampled independently per pixel on each frame.
-               That pixel's noise value is added to each of its color
-               channels, which at that point lie in the range [0,1]. -->
-          <mean>0.0</mean>
-          <stddev>0.007</stddev>
-        </noise>
-      </camera>
-      <plugin name="camera_controller" filename="libgazebo_ros_camera.so">
-        <alwaysOn>true</alwaysOn>
-        <updateRate>0.0</updateRate>
-        <cameraName>rrbot/camera1</cameraName>
-        <imageTopicName>image_raw</imageTopicName>
-        <cameraInfoTopicName>camera_info</cameraInfoTopicName>
-        <frameName>camera_link</frameName>
-        <hackBaseline>0.07</hackBaseline>
-        <distortionK1>0.0</distortionK1>
-        <distortionK2>0.0</distortionK2>
-        <distortionK3>0.0</distortionK3>
-        <distortionT1>0.0</distortionT1>
-        <distortionT2>0.0</distortionT2>
-      </plugin>
-    </sensor>
+    <plugin name="p3d_base_controller" filename="libgazebo_ros_p3d.so">
+      <alwaysOn>true</alwaysOn>
+      <updateRate>50.0</updateRate>
+      <bodyName>base_link</bodyName>
+      <topicName>ground_truth_pose</topicName>
+      <gaussianNoise>0.0</gaussianNoise>
+      <frameName>world</frameName>
+      <xyzOffsets>0 0 0</xyzOffsets>
+      <rpyOffsets>0 0 0</rpyOffsets>
+    </plugin>
   </gazebo>
 </robot>

File: src/go_car_description/urdf/include/links.xacro (robot description, xacro)
@@ -62,14 +62,4 @@
     </xacro:macro>
     <link name="camera_link">
-        <collision>
-            <geometry>
-                <box size="0.5 0.5 0.5"/>
-            </geometry>
-        </collision>
-        <visual>
-            <geometry>
-                <box size="0.5 0.5 0.5"/>
-            </geometry>
-        </visual>
         <inertial>
             <mass value="0.25"/>
@@ -78,14 +68,4 @@
     </link>
     <link name="lidar_link">
-        <collision>
-            <geometry>
-                <cylinder radius="0.1" length="0.2"/>
-            </geometry>
-        </collision>
-        <visual>
-            <geometry>
-                <cylinder radius="0.1" length="0.2"/>
-            </geometry>
-        </visual>
         <inertial>
             <mass value="0.25"/>

Commit message: feature: functional navigation package

File: src/go_car_description/urdf/go_car_model.xacro (robot description, xacro)
@@ -70,5 +70,5 @@
     <parent link="chassis_link"/>
     <child link="lidar_link"/>
-    <origin xyz="${chassis_length/2+0.25} 0.0 -0.25" rpy="0.0 0.0 0.0"/>
+    <origin xyz="0.0 0.0 0.9" rpy="0.0 0.0 0.0"/>
   </joint>
   <!-- Gazebo -->

File: src/go_car_description/urdf/include/sensors.xacro (robot description, xacro)
@@ -50,6 +50,6 @@
                         <samples>720</samples>
                         <resolution>1</resolution>
-                        <min_angle>-1.570796</min_angle>
-                        <max_angle>1.570796</max_angle>
+                        <min_angle>-3.14</min_angle>
+                        <max_angle>3.14</max_angle>
                     </horizontal>
                     <vertical>
@@ -61,6 +61,6 @@
                 </scan>
                 <range>
-                    <min>0.3</min>
-                    <max>131.0</max>
+                    <min>1.0</min>
+                    <max>130.0</max>
                     <resolution>0.001</resolution>
                 </range>
@@ -68,5 +68,5 @@
                     <type>gaussian</type>
                     <mean>0.0</mean>
-                    <stddev>0.0</stddev>
+                    <stddev>0.008</stddev>
                 </noise>
             </ray>
@@ -75,5 +75,5 @@
                 <frameName>lidar_link</frameName>
                 <organize_cloud>false</organize_cloud>
-                <min_range>0.9</min_range>
+                <min_range>1.0</min_range>
                 <max_range>130.0</max_range>
                 <gaussianNoise>0.008</gaussianNoise>

Commit message: feature: hdl32e specifications applied to 3d lidar

File: src/go_car_description/urdf/go_car_model.xacro (robot description, xacro)
@@ -65,10 +65,10 @@
     <parent link="chassis_link"/>
     <child link="camera_link"/>
-    <origin xyz="0.0 0.0 0.8" rpy="0.0 0.0 0.0"/>
+    <origin xyz="0.5 0.0 ${camera_height}" rpy="0.0 0.0 0.0"/>
   </joint>
   <joint name="chassis_to_lidar" type="fixed">
     <parent link="chassis_link"/>
     <child link="lidar_link"/>
-    <origin xyz="0.0 0.0 0.9" rpy="0.0 0.0 0.0"/>
+    <origin xyz="0.0 0.0 ${lidar_height}" rpy="0.0 0.0 0.0"/>
   </joint>
   <!-- Gazebo -->

File: src/go_car_description/urdf/include/links.xacro (robot description, xacro)
@@ -66,4 +66,10 @@
             <inertia ixx="1e-3" ixy="0" ixz="0" iyy="1e-3" iyz="0" izz="1e-3"/>
         </inertial>
+        <visual>
+            <origin xyz="0.0 -0.2 0.0" rpy="0.0 0.0 ${pi/2}"/>
+            <geometry>
+                <mesh filename="package://go_car_description/meshes/intel_realsense_camera.dae" scale="4.0 4.0 4.0"/>
+            </geometry>
+        </visual>
     </link>
     <link name="lidar_link">
@@ -72,4 +78,16 @@
             <inertia ixx="1e-3" ixy="0" ixz="0" iyy="1e-3" iyz="0" izz="1e-3"/>
         </inertial>
+        <visual>
+            <origin xyz="0.0 0.0 0.0" rpy="0.0 0.0 ${pi/2}"/>
+            <geometry>
+                <mesh filename="package://go_car_description/meshes/hdl32e.dae" scale="2.5 2.5 2.5"/>
+            </geometry>
+        </visual>
+        <visual>
+            <origin xyz="0.0 0.0 -0.4" rpy="0.0 0.0 0.0"/>
+            <geometry>
+                <mesh filename="package://go_car_description/meshes/hdl32e_base.dae" scale="2.5 2.5 7.5"/>
+            </geometry>
+        </visual>
     </link>
 </robot>

File: src/go_car_description/urdf/include/params.xacro (robot description, xacro)
@@ -52,3 +52,6 @@
     <xacro:property name="tyre_radius" value="0.356"/>
     <xacro:property name="tyre_width" value="0.229"/>
+    <!-- Sensors location setup params -->
+    <xacro:property name="lidar_height" value="1.0"/>
+    <xacro:property name="camera_height" value="0.625"/>
 </robot>

File: src/go_car_description/urdf/include/sensors.xacro (robot description, xacro)
@@ -2,5 +2,5 @@
 <robot xmlns:xacro="gazebo_sensors">
     <gazebo reference="camera_link">
-        <sensor type="camera" name="camera1">
+        <sensor type="camera" name="camera">
             <update_rate>30.0</update_rate>
             <camera name="head">
@@ -44,29 +44,29 @@
             <pose>0 0 0 0 0 0</pose>
             <visualize>false</visualize>
-            <update_rate>10</update_rate>
+            <update_rate>5</update_rate>
             <ray>
                 <scan>
                     <horizontal>
-                        <samples>720</samples>
+                        <samples>300</samples>                        <!-- Real sensor will have up to 1200 -->
                         <resolution>1</resolution>
-                        <min_angle>-3.14</min_angle>
-                        <max_angle>3.14</max_angle>
+                        <min_angle>${-pi}</min_angle>
+                        <max_angle>${pi}</max_angle>
                     </horizontal>
                     <vertical>
-                        <samples>32</samples>
+                        <samples>40</samples>
                         <resolution>1</resolution>
-                        <min_angle>-${30.67*1.570796/180.0}</min_angle>
-                        <max_angle> ${10.67*1.570796/180.0}</max_angle>
+                        <min_angle>${-30*pi/180}</min_angle>
+                        <max_angle>${10*pi/180}</max_angle>
                     </vertical>
                 </scan>
                 <range>
-                    <min>1.0</min>
-                    <max>130.0</max>
-                    <resolution>0.001</resolution>
+                    <min>3.0</min>
+                    <max>100.0</max>
+                    <resolution>0.005</resolution>
                 </range>
                 <noise>
                     <type>gaussian</type>
                     <mean>0.0</mean>
-                    <stddev>0.008</stddev>
+                    <stddev>0.02</stddev>
                 </noise>
             </ray>
@@ -75,7 +75,7 @@
                 <frameName>lidar_link</frameName>
                 <organize_cloud>false</organize_cloud>
-                <min_range>1.0</min_range>
-                <max_range>130.0</max_range>
-                <gaussianNoise>0.008</gaussianNoise>
+                <min_range>3.0</min_range>
+                <max_range>100.0</max_range>
+                <gaussianNoise>0.02</gaussianNoise>
             </plugin>
         </sensor>
