Commit message: version: prerelease

File: src/go_car_description/urdf/go_car_model.xacro (robot description, xacro)
@@ -7,9 +7,8 @@
   <xacro:include filename="$(find go_car_description)/urdf/include/sensors.xacro"/>
   <!-- First tf level -->
-  <link name="base_link"/>
   <joint name="base_to_chassis" type="fixed">
-    <parent link="base_link"/>
+    <parent link="base_footprint_link"/>
     <child link="chassis_link"/>
-    <origin xyz="0.0 0.0 0.0" rpy="0.0 0.0 0.0"/>
+    <origin xyz="0.0 0.0 0.84" rpy="0.0 0.0 0.0"/>
   </joint>
   <joint name="chassis_to_left_steering_column" type="revolute">
@@ -72,4 +71,24 @@
     <origin xyz="0.0 0.0 ${lidar_height}" rpy="0.0 0.0 0.0"/>
   </joint>
+  <joint name="chassis_to_back_ultrasonic" type="fixed">
+    <parent link="chassis_link"/>
+    <child link="back_ultrasonic_link"/>
+    <origin xyz="${-chassis_length/2} 0.0 0.0" rpy="0.0 0.0 ${pi}"/>
+  </joint>
+  <joint name="chassis_to_right_ultrasonic" type="fixed">
+    <parent link="chassis_link"/>
+    <child link="right_ultrasonic_link"/>
+    <origin xyz="0.0 ${-chassis_width/2} 0.0" rpy="0.0 0.0 ${-pi/2}"/>
+  </joint>
+  <joint name="chassis_to_left_ultrasonic" type="fixed">
+    <parent link="chassis_link"/>
+    <child link="left_ultrasonic_link"/>
+    <origin xyz="0.0 ${chassis_width/2} 0.0" rpy="0.0 0.0 ${pi/2}"/>
+  </joint>
+  <joint name="chassis_to_front_ultrasonic" type="fixed">
+    <parent link="chassis_link"/>
+    <child link="front_ultrasonic_link"/>
+    <origin xyz="${chassis_length/2+0.35} 0.0 0.0" rpy="0.0 0.0 0.0"/>
+  </joint>
   <!-- Gazebo -->
   <xacro:include filename="$(find go_car_description)/urdf/include/gazebo.xacro"/>

File: src/go_car_description/urdf/include/gazebo.xacro (robot description, xacro)
@@ -71,5 +71,5 @@
       <alwaysOn>true</alwaysOn>
       <updateRate>50.0</updateRate>
-      <bodyName>base_link</bodyName>
+      <bodyName>base_footprint_link</bodyName>
       <topicName>ground_truth_pose</topicName>
       <gaussianNoise>0.0</gaussianNoise>

File: src/go_car_description/urdf/include/links.xacro (robot description, xacro)
@@ -1,4 +1,5 @@
 <?xml version="1.0"?>
 <robot xmlns:xacro="properties_xacro">
+    <link name="base_footprint_link"/>
     <xacro:macro name="chassis_link" params="details">
         <link name="chassis_link">
@@ -91,3 +92,7 @@
         </visual>
     </link>
+    <link name="back_ultrasonic_link"/>
+    <link name="right_ultrasonic_link"/>
+    <link name="left_ultrasonic_link"/>
+    <link name="front_ultrasonic_link"/>
 </robot>

File: src/go_car_description/urdf/include/sensors.xacro (robot description, xacro)
@@ -74,5 +74,5 @@
                 <topicName>velodyne_points</topicName>
                 <frameName>lidar_link</frameName>
-                <organize_cloud>false</organize_cloud>
+                <organize_cloud>true</organize_cloud>
                 <min_range>3.0</min_range>
                 <max_range>100.0</max_range>
@@ -84,5 +84,5 @@
         <plugin name="navsat_sensor" filename="libhector_gazebo_ros_gps.so">
             <updateRate>1.0</updateRate>
-            <bodyName>base_link</bodyName>
+            <bodyName>chassis_link</bodyName>
             <topicName>/gps/coordinates</topicName>
             <velocityTopicName>/gps/velocity</velocityTopicName>
@@ -98,5 +98,5 @@
         <sensor type="lidar" name="liDAR_2d">
             <pose>0 0 0 0 0 0</pose>
-            <visualize>true</visualize>
+            <visualize>false</visualize>
             <update_rate>20</update_rate>
             <ray>
@@ -126,22 +126,169 @@
         </sensor>
     </gazebo> -->
-    <gazebo reference="base_link">
+    <gazebo reference="chassis_link">
         <gravity>true</gravity>
         <sensor name="imu_sensor" type="imu">
             <always_on>true</always_on>
             <update_rate>100</update_rate>
-            <visualize>true</visualize>
+            <visualize>false</visualize>
             <topic>__default_topic__</topic>
             <plugin filename="libgazebo_ros_imu_sensor.so" name="imu_plugin">
                 <topicName>imu</topicName>
-                <bodyName>base_link</bodyName>
+                <bodyName>chassis_link</bodyName>
                 <updateRateHZ>10.0</updateRateHZ>
                 <gaussianNoise>0.0</gaussianNoise>
                 <xyzOffset>0 0 0</xyzOffset>
                 <rpyOffset>0 0 0</rpyOffset>
-                <frameName>base_link</frameName>
-                <initialOrientationAsReference>false</initialOrientationAsReference>
-            </plugin>
-            <pose>0 0 0 0 0 0</pose>
+                <frameName>chassis_link</frameName>
+            </plugin>
+            <pose>0 0 0 0 0 0</pose>
+        </sensor>
+    </gazebo>
+    <gazebo reference="front_ultrasonic_link">
+        <sensor type="ray" name="TeraRanger">
+            <pose>0 0 0 0 0 0</pose>
+            <visualize>false</visualize>
+            <update_rate>50</update_rate>
+            <ray>
+                <scan>
+                    <horizontal>
+                        <samples>10</samples>
+                        <resolution>1</resolution>
+                        <min_angle>-0.14835</min_angle>
+                        <max_angle>0.14835</max_angle>
+                    </horizontal>
+                    <vertical>
+                        <samples>10</samples>
+                        <resolution>1</resolution>
+                        <min_angle>-0.14835</min_angle>
+                        <max_angle>0.14835</max_angle>
+                    </vertical>
+                </scan>
+                <range>
+                    <min>0.01</min>
+                    <max>2</max>
+                    <resolution>0.02</resolution>
+                </range>
+            </ray>
+            <plugin filename="libgazebo_ros_range.so" name="gazebo_ros_range">
+                <gaussianNoise>0.005</gaussianNoise>
+                <alwaysOn>true</alwaysOn>
+                <updateRate>50</updateRate>
+                <topicName>range_sensor/front</topicName>
+                <frameName>front_ultrasonic_link</frameName>
+                <radiation>INFRARED</radiation>
+                <fov>0.2967</fov>
+            </plugin>
+        </sensor>
+    </gazebo>
+    <gazebo reference="back_ultrasonic_link">
+        <sensor type="ray" name="TeraRanger">
+            <pose>0 0 0 0 0 0</pose>
+            <visualize>false</visualize>
+            <update_rate>50</update_rate>
+            <ray>
+                <scan>
+                    <horizontal>
+                        <samples>10</samples>
+                        <resolution>1</resolution>
+                        <min_angle>-0.14835</min_angle>
+                        <max_angle>0.14835</max_angle>
+                    </horizontal>
+                    <vertical>
+                        <samples>10</samples>
+                        <resolution>1</resolution>
+                        <min_angle>-0.14835</min_angle>
+                        <max_angle>0.14835</max_angle>
+                    </vertical>
+                </scan>
+                <range>
+                    <min>0.01</min>
+                    <max>2</max>
+                    <resolution>0.02</resolution>
+                </range>
+            </ray>
+            <plugin filename="libgazebo_ros_range.so" name="gazebo_ros_range">
+                <gaussianNoise>0.005</gaussianNoise>
+                <alwaysOn>true</alwaysOn>
+                <updateRate>50</updateRate>
+                <topicName>range_sensor/back</topicName>
+                <frameName>back_ultrasonic_link</frameName>
+                <radiation>INFRARED</radiation>
+                <fov>0.2967</fov>
+            </plugin>
+        </sensor>
+    </gazebo>
+    <gazebo reference="right_ultrasonic_link">
+        <sensor type="ray" name="TeraRanger">
+            <pose>0 0 0 0 0 0</pose>
+            <visualize>false</visualize>
+            <update_rate>50</update_rate>
+            <ray>
+                <scan>
+                    <horizontal>
+                        <samples>10</samples>
+                        <resolution>1</resolution>
+                        <min_angle>-0.14835</min_angle>
+                        <max_angle>0.14835</max_angle>
+                    </horizontal>
+                    <vertical>
+                        <samples>10</samples>
+                        <resolution>1</resolution>
+                        <min_angle>-0.14835</min_angle>
+                        <max_angle>0.14835</max_angle>
+                    </vertical>
+                </scan>
+                <range>
+                    <min>0.01</min>
+                    <max>2</max>
+                    <resolution>0.02</resolution>
+                </range>
+            </ray>
+            <plugin filename="libgazebo_ros_range.so" name="gazebo_ros_range">
+                <gaussianNoise>0.005</gaussianNoise>
+                <alwaysOn>true</alwaysOn>
+                <updateRate>50</updateRate>
+                <topicName>range_sensor/right</topicName>
+                <frameName>right_ultrasonic_link</frameName>
+                <radiation>INFRARED</radiation>
+                <fov>0.2967</fov>
+            </plugin>
+        </sensor>
+    </gazebo>
+    <gazebo reference="left_ultrasonic_link">
+        <sensor type="ray" name="TeraRanger">
+            <pose>0 0 0 0 0 0</pose>
+            <visualize>false</visualize>
+            <update_rate>50</update_rate>
+            <ray>
+                <scan>
+                    <horizontal>
+                        <samples>10</samples>
+                        <resolution>1</resolution>
+                        <min_angle>-0.14835</min_angle>
+                        <max_angle>0.14835</max_angle>
+                    </horizontal>
+                    <vertical>
+                        <samples>10</samples>
+                        <resolution>1</resolution>
+                        <min_angle>-0.14835</min_angle>
+                        <max_angle>0.14835</max_angle>
+                    </vertical>
+                </scan>
+                <range>
+                    <min>0.01</min>
+                    <max>2</max>
+                    <resolution>0.02</resolution>
+                </range>
+            </ray>
+            <plugin filename="libgazebo_ros_range.so" name="gazebo_ros_range">
+                <gaussianNoise>0.005</gaussianNoise>
+                <alwaysOn>true</alwaysOn>
+                <updateRate>50</updateRate>
+                <topicName>range_sensor/left</topicName>
+                <frameName>left_ultrasonic_link</frameName>
+                <radiation>INFRARED</radiation>
+                <fov>0.2967</fov>
+            </plugin>
         </sensor>
     </gazebo>
